File: VooDoo 4x PCIe.kicad_pcb (KiCad board)
At the start: 4 copper layers, 122.7 x 111.2 mm, 107 parts, among them CN1 HF1004E, IC1 BM1397_mode1, J1 PCIexpress_x1, J2 USB_C_Receptacle_USB2.0, J3 Conn_01x05, Q1 CSD17551Q3A, Q2 CSD17575Q3, U1 TPS40305, U10 FT230XQ, U2 LN1134A182MR-G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

Commit message: Voodoo Miner X1 WIP
Updated Nets and base routing is 99% done
Routing:
- net /Asic/1V8: track 86.1 -> 103.5 mm, vias 3 -> 5
- net TEMP_P: track 39.8 -> 50.6 mm
- net /Asic/0V8: track 22.7 -> 26.1 mm
- net 5V: track 97.4 -> 95.3 mm
- net GND: track 142.2 -> 143.4 mm, vias 105 -> 106
